File: GECW/GCEW/GCEW.sch (KiCad schematic (older format))
At the start: 35 parts, among them Q1 Q_NMOS_DGS, Q2 Q_NMOS_DGS, Q3 Q_NMOS_DGS, Q4 Q_NMOS_DGS, Q5 Q_NMOS_DGS, Q6 Q_NMOS_DGS, U1 DRV8323RHRGZ, U2 BLDCMOTOR

Commit message: Schematic is dramatic
Cleaned and updated schematic
Parts:
- added C9: 4.7uF, symbol Device:C
- added MCU1: Conn_01x07_Male, symbol Connector:Conn_01x07_Male
- added U3: LM26CIM5-VHA, symbol myLib:LM26CIM5-VHA
- C10: renamed from C8; footprint (none) -> Capacitor_SMD:C_0805_2012Metric
- R1, R10, R11, R12, R13, R14, R2, R3, R5, R6, R8, R9: footprint (none) -> Resistor_SMD:R_1206_3216Metric
- R4, R7: value 600k -> 1M; footprint (none) -> Resistor_SMD:R_1206_3216Metric
- U1: footprint RGZ0048A -> (none)
- renumbered C6 to C1, C7 to C11, C5 to C2, C4 to C3, C9 to C4, C1 to C5, C2 to C6, C3 to C7, C10 to C8, 36V1 to VDC1
Connections:
- net labels added: +5V, CAL, H_A, H_B, H_C, INHA, INHC, INLC, SOA, SOB, SOC, Vtemp
- net labels removed: GNDD, GNDPWR
- wire segments 180 -> 166
